Commit message: fix the origin of the collision box for the head

File: hlpr_poli/poli_description/urdf/poli_neck_head.urdf.xacro (robot description, xacro)
@@ -81,7 +81,7 @@
           </visual>
           <collision>
-            <origin xyz="0 0 0" rpy="0 0 0" />
+            <origin xyz="0.01 -0.09 0" rpy="0 0 0" />
             <geometry>
-              <box size="0.32 0.2 0.35" />
+              <box size="0.33 0.18 0.37" />
             </geometry>
           </collision>

Commit message: added in the experimentally verified limits for the pan and tilt joints

File: hlpr_poli/poli_description/urdf/poli_neck_head.urdf.xacro (robot description, xacro)
@@ -21,5 +21,5 @@
             <child link="pan_link" />
             <axis xyz="0 0 1"/>
-            <limit effort="6.0" lower="-0.523599" upper="0.523599" velocity="6.597"/>
+            <limit effort="6.0" lower="-0.75" upper="0.75" velocity="6.597"/>
         </joint>
         <link name="pan_link">
@@ -56,5 +56,5 @@
           <child link="tilt_link" />
           <axis xyz="0 0 1" />
-          <limit effort="6.0" lower="-0.174533" upper="0.785398" velocity="6.597"/>
+          <limit effort="6.0" lower="-0.25" upper="0.589" velocity="6.597"/>
         </joint>
         <link name="tilt_link">
