Commit message: updated poli urdf to take into account the basket

File: hlpr_poli/poli_description/urdf/basket.urdf.xacro (robot description, xacro)
@@ -21,4 +21,7 @@
                         <box size="0.14 0.275 0.165"/>
                     </geometry>
+                    <material name="">
+                      <color rgba="0.75294 0.75294 0.75294 1" />
+                    </material>
                 </visual>
             </xacro:if>
