Commit message: tested poli launch with pan tilt and linear actuator controllers. Also set soft limits for the linear actuator. Current pan tilt limits are not accurate

File: hlpr_poli/poli_description/robots/poli.urdf.xacro (robot description, xacro)
@@ -110,3 +110,4 @@
         <origin xyz="0 0 0.131" rpy="0 0 0"/>
     </xacro:poli_neck_head>
+    <xacro:poli_neck_head_transmission/>
 </robot>

File: hlpr_poli/poli_description/urdf/poli_linear_actuator_neck.urdf.xacro (robot description, xacro)
@@ -42,5 +42,5 @@
           <child link="linear_actuator_link" />
           <axis xyz="0 0 1" />
-          <limit lower="0.0" upper="0.855" effort="1000" velocity="0.20"/>
+          <limit lower="0.0" upper="0.70" effort="1000" velocity="0.20"/>
           <dynamics damping="0.0" friction="0.0"/>
         </joint>

File: hlpr_poli/poli_description/urdf/poli_neck_head.transmission.xacro (robot description, xacro)
@@ -2,19 +2,19 @@
 <robot xmlns:xacro="http://www.ros.org/wiki/xacro">
   <xacro:macro name="poli_neck_head_transmission">
-    <transmission name="head_yaw_trans">
+    <transmission name="pan_trans">
       <type>transmission_interface/SimpleTransmission</type>
-      <joint name="head_yaw_joint">
+      <joint name="pan_joint">
         <hardwareInterface>PositionJointInterface</hardwareInterface>
       </joint>
-      <actuator name="head_yaw_motor">
+      <actuator name="pan_motor">
         <mechanicalReduction>1</mechanicalReduction>
       </actuator>
     </transmission>
-    <transmission name="head_pitch_trans">
+    <transmission name="tilt_trans">
       <type>transmission_interface/SimpleTransmission</type>
-      <joint name="head_pitch_joint">
+      <joint name="tilt_joint">
         <hardwareInterface>PositionJointInterface</hardwareInterface>
       </joint>
-      <actuator name="head_pitch_motor">
+      <actuator name="tilt_motor">
         <mechanicalReduction>1</mechanicalReduction>
       </actuator>

File: hlpr_poli/poli_description/urdf/poli_neck_head.urdf.xacro (robot description, xacro)
@@ -2,12 +2,12 @@
 <robot xmlns:xacro="http://ros.org/wiki/xacro" name="poli_neck_head">
     <xacro:macro name="poli_neck_head" params="parent *origin">
-        <joint name="head_yaw_joint" type="revolute">
+        <joint name="pan_joint" type="revolute">
             <xacro:insert_block name="origin" />
             <parent link="${parent}" />
-            <child link="head_yaw" />
+            <child link="pan_link" />
             <axis xyz="0 0 1"/>
-            <limit effort="0" velocity="0"/>
+            <limit effort="6.0" lower="-1.570796326794897" upper="1.570796326794897" velocity="6.597"/>
         </joint>
-        <link name="head_yaw">
+        <link name="pan_link">
           <inertial>
             <origin xyz="-0.00051082 4.6611E-05 -0.0079247" rpy="0 0 0" />
@@ -37,5 +37,5 @@
           </collision>
         </link>
-        <link name="head_pitch">
+        <link name="tilt_link">
           <inertial>
             <origin xyz="0.061895 -0.074515 0.00018285" rpy="0 0 0" />
@@ -65,10 +65,10 @@
           </collision>
         </link>
-        <joint name="head_pitch_joint" type="revolute">
+        <joint name="tilt_joint" type="revolute">
           <origin xyz="0 0 0" rpy="-1.5708 0 0" />
-          <parent link="head_yaw" />
-          <child link="head_pitch" />
-          <axis xyz="0 0 -1" />
-          <limit effort="0" velocity="0" />
+          <parent link="pan_link" />
+          <child link="tilt_link" />
+          <axis xyz="0 0 1" />
+          <limit effort="6.0" lower="-1.047197551196598" upper="1.570796326794897" velocity="6.597"/>
         </joint>
     </xacro:macro>

Commit message: fixed to include lasers on the robot with the correct laser distance

File: hlpr_poli/poli_description/robots/poli.urdf.xacro (robot description, xacro)
@@ -28,6 +28,10 @@
     <xacro:include filename="$(find poli_description)/urdf/poli_linear_actuator_neck.urdf.xacro" />
     <xacro:include filename="$(find poli_description)/urdf/poli_neck_head.urdf.xacro" />
+    <!-- Include sensor files -->
+    <xacro:include filename="$(find vector_description)/urdf/sensors/kinect_one_sensor.urdf.xacro" />
+    <xacro:include filename="$(find poli_description)/urdf/laser_sensors.urdf.xacro" />
     <!-- Include transmission Files -->
     <xacro:include filename="$(find poli_description)/urdf/poli_neck_head.transmission.xacro" />
+    <!-- Robot base -->
     <xacro:property name="M_PI" value="3.14159"/>
     <xacro:if value="$(optenv VECTOR_USE_PLATFORM_ODOMETRY false)">
@@ -111,3 +115,9 @@
     </xacro:poli_neck_head>
     <xacro:poli_neck_head_transmission/>
+    <!-- include the kinect sensor -->
+    <xacro:kinect_one_sensor prefix="kinect" parent="tilt_link">
+       <origin xyz="0.1125 -0.03425 0" rpy="${M_PI/2} 0 0" />
+    </xacro:kinect_one_sensor>
+    <!-- Include the lasers -->
+    <xacro:poli_lasers />
 </robot>

File: hlpr_poli/poli_description/urdf/poli_linear_actuator_neck.urdf.xacro (robot description, xacro)
@@ -9,8 +9,11 @@
 	    <link name="linear_actuator_fixed_link">
 			<visual>
-                <origin xyz="0 0 0" rpy="0 0 0"/>
+			    <origin xyz="0 0 0" rpy="0 0 0"/>
 				  <geometry>
 					<mesh filename="package://poli_description/meshes/base_link.STL" />
 				</geometry>
+				  <material name="">
+				      <color rgba="0.75294 0.75294 0.75294 1" />
+				  </material>
 			</visual>
 			<collision>

Commit message: add conservative limits to neck and add in pan_base_link

File: hlpr_poli/poli_description/robots/poli.urdf.xacro (robot description, xacro)
@@ -112,5 +112,5 @@
     </xacro:poli_linear_actuator>
     <xacro:poli_neck_head parent="linear_actuator_fixed_link">
-        <origin xyz="0 0 0.131" rpy="0 0 0"/>
+        <origin xyz="0 0 0" rpy="0 0 0"/>
     </xacro:poli_neck_head>
     <xacro:poli_neck_head_transmission/>

File: hlpr_poli/poli_description/urdf/poli_neck_head.urdf.xacro (robot description, xacro)
@@ -2,10 +2,24 @@
 <robot xmlns:xacro="http://ros.org/wiki/xacro" name="poli_neck_head">
     <xacro:macro name="poli_neck_head" params="parent *origin">
-        <joint name="pan_joint" type="revolute">
+        <joint name="pan_base_joint" type="fixed">
             <xacro:insert_block name="origin" />
             <parent link="${parent}" />
+            <child link="pan_base_link" />
+        </joint>
+        <link name="pan_base_link">
+            <inertial>
+                <mass value="0.1"/>
+                <origin xyz="0 0 0" rpy="0 0 0"/>
+                <inertia ixx="0.01"  ixy="0.0"  ixz="0.0"
+                         iyy="0.01"  iyz="0.0"
+                         izz="0.01" />
+            </inertial>
+        </link>
+        <joint name="pan_joint" type="revolute">
+            <origin xyz="0 0 0.131" rpy="0 0 0" />
+            <parent link="pan_base_link" />
             <child link="pan_link" />
             <axis xyz="0 0 1"/>
-            <limit effort="6.0" lower="-1.570796326794897" upper="1.570796326794897" velocity="6.597"/>
+            <limit effort="6.0" lower="-0.523599" upper="0.523599" velocity="6.597"/>
         </joint>
         <link name="pan_link">
@@ -37,4 +51,11 @@
           </collision>
         </link>
+        <joint name="tilt_joint" type="revolute">
+          <origin xyz="0 0 0" rpy="-1.570796326794897 0 0" />
+          <parent link="pan_link" />
+          <child link="tilt_link" />
+          <axis xyz="0 0 1" />
+          <limit effort="6.0" lower="-0.174533" upper="0.785398" velocity="6.597"/>
+        </joint>
         <link name="tilt_link">
           <inertial>
@@ -65,11 +86,4 @@
           </collision>
         </link>
-        <joint name="tilt_joint" type="revolute">
-          <origin xyz="0 0 0" rpy="-1.5708 0 0" />
-          <parent link="pan_link" />
-          <child link="tilt_link" />
-          <axis xyz="0 0 1" />
-          <limit effort="6.0" lower="-1.047197551196598" upper="1.570796326794897" velocity="6.597"/>
-        </joint>
     </xacro:macro>
 </robot>

Commit message: newest versions of urdf with body shell and simplified collisions bodies

File: hlpr_poli/poli_description/robots/poli.urdf.xacro (robot description, xacro)
@@ -28,4 +28,5 @@
     <xacro:include filename="$(find poli_description)/urdf/poli_linear_actuator_neck.urdf.xacro" />
     <xacro:include filename="$(find poli_description)/urdf/poli_neck_head.urdf.xacro" />
+    <xacro:include filename="$(find poli_description)/urdf/poli_body.urdf.xacro" />
     <!-- Include sensor files -->
     <xacro:include filename="$(find vector_description)/urdf/sensors/kinect_one_sensor.urdf.xacro" />
@@ -72,10 +73,4 @@
     </xacro:unless>
     <xacro:vector_base name="base"/>
-    <!--linear actuator-->
-    <xacro:if value="$(optenv VECTOR_HAS_LINEAR_ACTUATOR true)">
-        <xacro:vector_linear_actuator parent="base_chassis_link">
-            <origin xyz="0.22806971 0 0.46024800" rpy="0 0 0" />
-        </xacro:vector_linear_actuator>
-    </xacro:if>
     <!-- Arms -->
     <xacro:if value="$(optenv VECTOR_HAS_KINOVA_ARM false)">
@@ -111,4 +106,8 @@
         <origin xyz="0.2015 0 1.3642" rpy="0 0 0" />
     </xacro:poli_linear_actuator>
+    <!-- Poli's coat -->
+    <xacro:poli_body parent="base_chassis_link">
+        <origin xyz="0 0 0" rpy="0 0 -${M_PI/2}" />
+    </xacro:poli_body>
     <xacro:poli_neck_head parent="linear_actuator_fixed_link">
         <origin xyz="0 0 0" rpy="0 0 0"/>

File: hlpr_poli/poli_description/urdf/poli_linear_actuator_neck.urdf.xacro (robot description, xacro)
@@ -7,36 +7,32 @@
             <child link="linear_actuator_fixed_link" />
         </joint>
-	    <link name="linear_actuator_fixed_link">
-			<visual>
-			    <origin xyz="0 0 0" rpy="0 0 0"/>
-				  <geometry>
-					<mesh filename="package://poli_description/meshes/base_link.STL" />
-				</geometry>
-				  <material name="">
-				      <color rgba="0.75294 0.75294 0.75294 1" />
-				  </material>
-			</visual>
-			<collision>
-				<geometry>
-					<mesh filename="package://poli_description/meshes/base_link.STL" />
-				</geometry>
-			</collision>
+	<link name="linear_actuator_fixed_link">
+		<visual>
+		    <origin xyz="0 0 0" rpy="0 0 0"/>
+  		    <geometry>
+			<mesh filename="package://poli_description/meshes/base_link.STL" />
+		    </geometry>
+		    <material name="">
+		      <color rgba="0.75294 0.75294 0.75294 1" />
+		    </material>
+		</visual>
+		<collision>
+			<origin xyz="0 0 -0.485" rpy="0 0 0"/>
+			<geometry>
+			    <box size="0.09 0.09 1.2" />
+			</geometry>
+		</collision>
             <inertial>
-              <origin xyz="-0.011801 0.024796 -0.63503" rpy="0 0 0" />
+              <origin xyz="-0.011319 0.023009 -0.586408" rpy="0 0 0" />
               <mass value="19.332" />
               <inertia
-                ixx="2.4716"
-                ixy="-0.0011724"
-                ixz="0.0085341"
-                iyy="2.4326"
-                iyz="-0.17433"
-                izz="0.066996" />
+                ixx="0.000398"
+                ixy="0.0"
+                ixz="-0.000002"
+                iyy="0.000393"
+                iyz="0.000025"
+                izz="0.000009" />
             </inertial>
-		    <!--inertial>
-                <mass value="5.098044" />
-                <origin xyz="0.0 0.0 0.5" rpy="0 0 0"/>
-                <inertia ixx="0.02"  ixy="0.0"  ixz="1.0" iyy="-0.03"  iyz="-0.02" izz="0.0" />
-		    </inertial-->
-		</link>
+	</link>
         <joint name="linear_joint" type="prismatic">
           <!--origin xyz="0.038771 -0.000254 -0.10409" rpy="0 0 0" /-->

File: hlpr_poli/poli_description/urdf/poli_neck_head.urdf.xacro (robot description, xacro)
@@ -47,5 +47,5 @@
             <origin xyz="0 0 0" rpy="0 0 0" />
             <geometry>
-              <mesh filename="package://poli_description/meshes/Yaw.STL" />
+              <box size="0.04 0.085 0.14" />
             </geometry>
           </collision>
@@ -60,5 +60,6 @@
         <link name="tilt_link">
           <inertial>
-            <origin xyz="0.061895 -0.074515 0.00018285" rpy="0 0 0" />
+            <!--origin xyz="0.061895 -0.074515 0.00018285" rpy="0 0 0" /-->
+            <origin xyz="0 -0.074515 0.00018285" rpy="0 0 0" />
             <mass value="1.6753" />
             <inertia
@@ -82,5 +83,5 @@
             <origin xyz="0 0 0" rpy="0 0 0" />
             <geometry>
-              <mesh filename="package://poli_description/meshes/Pitch.STL" />
+              <box size="0.32 0.2 0.35" />
             </geometry>
           </collision>

Commit message: added in astra camera and basket to URDF

File: hlpr_poli/poli_description/robots/poli.urdf.xacro (robot description, xacro)
@@ -29,7 +29,9 @@
     <xacro:include filename="$(find poli_description)/urdf/poli_neck_head.urdf.xacro" />
     <xacro:include filename="$(find poli_description)/urdf/poli_body.urdf.xacro" />
+    <xacro:include filename="$(find poli_description)/urdf/basket.urdf.xacro" />
     <!-- Include sensor files -->
     <xacro:include filename="$(find vector_description)/urdf/sensors/kinect_one_sensor.urdf.xacro" />
     <xacro:include filename="$(find poli_description)/urdf/laser_sensors.urdf.xacro" />
+    <xacro:include filename="$(find poli_description)/urdf/astra.urdf.xacro" />
     <!-- Include transmission Files -->
     <xacro:include filename="$(find poli_description)/urdf/poli_neck_head.transmission.xacro" />
@@ -101,5 +103,4 @@
     </xacro:if>
     <!-- Setup any accessories defined in the environment -->
-    <!--xacro:vector_accessories /-->
     <xacro:poli_linear_actuator parent="base_chassis_link">
         <!--origin xyz="0.22806971 0 0.46024800" rpy="0 0 0" /-->
@@ -120,3 +121,14 @@
     <!-- Include the lasers -->
     <xacro:poli_lasers />
+    <!-- Include the new RGBD Astra -->
+    <xacro:sensor_astra parent="base_chassis_link">
+       <origin xyz="0.30 -0.1 0.3125" rpy="0 0 0" />
+    </xacro:sensor_astra>
+    <!-- Include the basket -->
+    <xacro:basket number="1" parent="base_chassis_link" visual="true">
+       <origin xyz="0.34 0.1325 0.365" rpy="0 0 0" />
+    </xacro:basket>
+    <xacro:basket number="2" parent="base_chassis_link" visual="false">
+       <origin xyz="0.34 -0.1325 0.365" rpy="0 0 0" />
+    </xacro:basket>
 </robot>

Commit message: increase the size of the basket slightly for safety

File: hlpr_poli/poli_description/robots/poli.urdf.xacro (robot description, xacro)
@@ -127,8 +127,8 @@
     <!-- Include the basket -->
     <xacro:basket number="1" parent="base_chassis_link" visual="true">
-       <origin xyz="0.34 0.1325 0.365" rpy="0 0 0" />
+       <origin xyz="0.34 0.1325 0.37" rpy="0 0 0" />
     </xacro:basket>
     <xacro:basket number="2" parent="base_chassis_link" visual="false">
-       <origin xyz="0.34 -0.1325 0.365" rpy="0 0 0" />
+       <origin xyz="0.34 -0.1325 0.37" rpy="0 0 0" />
     </xacro:basket>
 </robot>

File: hlpr_poli/poli_description/urdf/basket.urdf.xacro (robot description, xacro)
@@ -19,5 +19,5 @@
                     <origin xyz="0 0 0" rpy="0 0 0"/>
                     <geometry>
-                        <box size="0.14 0.275 0.165"/>
+                        <box size="0.14 0.275 0.175"/>
                     </geometry>
                     <material name="">
@@ -29,5 +29,5 @@
                 <origin xyz="0 0 0" rpy="0 0 0"/>
                 <geometry>
-                    <box size="0.14 0.275 0.165"/>
+                    <box size="0.14 0.275 0.175"/>
                 </geometry>
             </collision>

Commit message: added sonar sensor

File: hlpr_poli/poli_description/robots/poli.urdf.xacro (robot description, xacro)
@@ -34,4 +34,5 @@
     <xacro:include filename="$(find poli_description)/urdf/laser_sensors.urdf.xacro" />
     <xacro:include filename="$(find poli_description)/urdf/astra.urdf.xacro" />
+    <xacro:include filename="$(find poli_description)/urdf/sonar.urdf.xacro" />
     <!-- Include transmission Files -->
     <xacro:include filename="$(find poli_description)/urdf/poli_neck_head.transmission.xacro" />
@@ -125,4 +126,8 @@
        <origin xyz="0.30 -0.1 0.3125" rpy="0 0 0" />
     </xacro:sensor_astra>
+    <!-- Include front sonar -->
+    <xacro:sensor_sonar parent="base_chassis_link">
+       <origin xyz="0.35 0.1 0.25" rpy="0 0 0" />
+    </xacro:sensor_sonar>
     <!-- Include the basket -->
     <xacro:basket number="1" parent="base_chassis_link" visual="true">
