Commit message: Fixed warnings about deprecated xacro syntax

File: hlpr_poli/poli_description/robots/poli_7dof.urdf.xacro (robot description, xacro)
@@ -79,7 +79,7 @@
     <xacro:if value="$(optenv VECTOR_HAS_KINOVA_ARM false)">
         <xacro:j2s7s300 base_parent="linear_actuator_link" trans="0.06079866 0 0" rot="${J_PI/2} 0 ${J_PI/2}">
-	    <!-- Note: origin is overwritten in kinova urdf -->
-            <origin xyz="0.06079866 0 0" rpy="${J_PI/2} 0 ${J_PI/2}" />
-	</xacro:j2s7s300>
+        <!-- Note: origin is overwritten in kinova urdf -->
+            <!-- <origin xyz="0.06079866 0 0" rpy="${J_PI/2} 0 ${J_PI/2}" /> -->
+        </xacro:j2s7s300>
     </xacro:if>
     <!-- Setup any accessories defined in the environment -->

File: hlpr_poli/poli_description/urdf/laser_sensors.urdf.xacro (robot description, xacro)
@@ -26,5 +26,5 @@
     <xacro:include filename="$(find poli_description)/urdf/hokuyo_ust30lx.urdf.xacro"/>
     <xacro:include filename="$(find poli_description)/urdf/hokuyo_ust10lx.urdf.xacro"/>
-    <property name="M_PI" value="3.14159"/>
+    <xacro:property name="M_PI" value="3.14159"/>
     <xacro:macro name="poli_lasers">
         <link name="sic_imu_frame"/>

File: hlpr_poli/poli_description/urdf/poli_neck_head.transmission.xacro (robot description, xacro)
@@ -1,4 +1,4 @@
 <?xml version="1.0"?>
-<robot xmlns:xacro="http://www.ros.org/wiki/xacro">
+<robot xmlns:xacro="http://ros.org/wiki/xacro">
   <xacro:macro name="poli_neck_head_transmission">
     <transmission name="pan_trans">
